Commit message: chore: fix bot geometry
Signed-off-by: Paulo Santos <prms@ic.ufal.br>

File: src/scara_robot_simulation/description/urdf/scara_rrrp.urdf.xacro (robot description, xacro)
@@ -1,19 +1,29 @@
 <?xml version="1.0"?>
 <robot xmlns:xacro="http://www.ros.org/wiki/xacro" name="scara_rrrp">
-    <gazebo reference="base_link">
-        <material>Gazebo/Grey</material>
-    </gazebo>
-    <gazebo reference="link1">
-        <material>Gazebo/Blue</material>
-    </gazebo>
-    <gazebo reference="link2">
-        <material>Gazebo/Red</material>
-    </gazebo>
-    <gazebo reference="link3">
-        <material>Gazebo/Blue</material>
-    </gazebo>
-    <gazebo reference="end_effector_link">
-        <material>Gazebo/Green</material>
-    </gazebo>
+    <xacro:property name="PI" value="3.1415926535897931"/>
+    <xacro:property name="base_height" value="0.5"/>
+    <xacro:property name="base_radius" value="0.04"/>
+    <xacro:property name="link1_length" value="0.3"/>
+    <xacro:property name="link2_length" value="0.2"/>
+    <xacro:property name="link_width" value="0.05"/>
+    <xacro:property name="link_height" value="0.05"/>
+    <xacro:property name="joint_housing_radius" value="0.03"/>
+    <xacro:property name="joint_housing_height" value="0.12"/>
+    <xacro:property name="quill_housing_length" value="0.1"/>
+    <xacro:property name="quill_housing_radius" value="0.03"/>
+    <xacro:property name="quill_length" value="0.25"/>
+    <xacro:property name="quill_radius" value="0.02"/>
+    <material name="light_grey">
+        <color rgba="0.7 0.7 0.7 1.0"/>
+    </material>
+    <material name="blue">
+        <color rgba="0.2 0.4 0.8 1.0"/>
+    </material>
+    <material name="black">
+        <color rgba="0.15 0.15 0.15 1.0"/>
+    </material>
+    <material name="chrome">
+        <color rgba="0.85 0.85 0.85 1.0"/>
+    </material>
     <link name="world"/>
     <joint name="world_to_base_joint" type="fixed">
@@ -25,17 +35,18 @@
         <visual>
             <geometry>
-                <cylinder length="1.0" radius="0.1"/>
-            </geometry>
-            <origin xyz="0 0 0.5" rpy="0 0 0"/>
-        </visual>
-        <collision>
-            <geometry>
-                <cylinder length="1.0" radius="0.1"/>
-            </geometry>
-            <origin xyz="0 0 0.5" rpy="0 0 0"/>
-        </collision>
-        <inertial>
-            <mass value="1.0"/>
-            <inertia ixx="0.1" ixy="0" ixz="0" iyy="0.1" iyz="0" izz="0.1"/>
+                <cylinder length="${base_height}" radius="${base_radius}"/>
+            </geometry>
+            <origin xyz="0 0 ${base_height/2}" rpy="0 0 0"/>
+            <material name="light_grey"/>
+        </visual>
+        <collision>
+            <geometry>
+                <cylinder length="${base_height}" radius="${base_radius}"/>
+            </geometry>
+            <origin xyz="0 0 ${base_height}" rpy="0 0 0"/>
+        </collision>
+        <inertial>
+            <mass value="5.0"/>
+            <inertia ixx="0.01" ixy="0" ixz="0" iyy="0.01" iyz="0" izz="0.02"/>
         </inertial>
     </link>
@@ -43,24 +54,33 @@
         <parent link="base_link"/>
         <child link="link1"/>
-        <origin xyz="0 0 1.0" rpy="0 0 0"/>
+        <origin xyz="0 0 ${base_height}" rpy="0 0 0"/>
         <axis xyz="0 0 1"/>
-        <limit lower="-3.14" upper="3.14" effort="10" velocity="1.0"/>
+        <limit lower="${-PI}" upper="${PI}" effort="100" velocity="1.0"/>
     </joint>
     <link name="link1">
         <visual>
             <geometry>
-                <box size="0.5 0.05 0.05"/>
-            </geometry>
-            <origin xyz="0.25 0 0" rpy="0 0 0"/>
-        </visual>
-        <collision>
-            <geometry>
-                <box size="0.5 0.05 0.05"/>
-            </geometry>
-            <origin xyz="0.25 0 0" rpy="0 0 0"/>
-        </collision>
-        <inertial>
-            <mass value="0.5"/>
-            <inertia ixx="0.1" ixy="0" ixz="0" iyy="0.1" iyz="0" izz="0.1"/>
+                <box size="${link1_length} ${link_width} ${link_height}"/>
+            </geometry>
+            <origin xyz="${link1_length/2} 0 ${link_width/2}" rpy="0 0 0"/>
+            <material name="blue"/>
+        </visual>
+        <collision>
+            <geometry>
+                <box size="${link1_length} ${link_width} ${link_height}"/>
+            </geometry>
+            <origin xyz="${link1_length/2} 0 0" rpy="0 0 0"/>
+        </collision>
+        <visual>
+            <geometry>
+                <cylinder radius="${joint_housing_radius}" length="${joint_housing_height}"/>
+            </geometry>
+            <origin xyz="0 0 0" rpy="0 0 0"/>
+            <material name="black"/>
+        </visual>
+        <inertial>
+            <mass value="1.5"/>
+            <origin xyz="${link1_length/2} 0 0" rpy="0 0 0"/>
+            <inertia ixx="0.01" ixy="0" ixz="0" iyy="0.01" iyz="0" izz="0.01"/>
         </inertial>
     </link>
@@ -68,75 +88,116 @@
         <parent link="link1"/>
         <child link="link2"/>
-        <origin xyz="0.5 0 0" rpy="0 0 0"/>
+        <origin xyz="${link1_length} 0 0" rpy="0 0 0"/>
         <axis xyz="0 0 1"/>
-        <limit lower="-2.5" upper="2.5" effort="10" velocity="1.0"/>
+        <limit lower="${-PI*0.8}" upper="${PI*0.8}" effort="100" velocity="1.0"/>
     </joint>
     <link name="link2">
         <visual>
             <geometry>
-                <box size="0.4 0.05 0.05"/>
-            </geometry>
-            <origin xyz="0.2 0 0" rpy="0 0 0"/>
-        </visual>
-        <collision>
-            <geometry>
-                <box size="0.4 0.05 0.05"/>
-            </geometry>
-            <origin xyz="0.2 0 0" rpy="0 0 0"/>
-        </collision>
-        <inertial>
-            <mass value="0.4"/>
-            <inertia ixx="0.1" ixy="0" ixz="0" iyy="0.1" iyz="0" izz="0.1"/>
-        </inertial>
-    </link>
-    <joint name="joint3" type="prismatic">
+                <box size="${link2_length} ${link_width} ${link_height}"/>
+            </geometry>
+            <origin xyz="${link2_length/2} 0 ${-link_height/2}" rpy="0 0 0"/>
+            <material name="blue"/>
+        </visual>
+        <collision>
+            <geometry>
+                <box size="${link2_length} ${link_width} ${link_height}"/>
+            </geometry>
+            <origin xyz="0 0 0" rpy="0 0 0"/>
+        </collision>
+        <visual>
+            <geometry>
+                <cylinder radius="${joint_housing_radius}" length="${joint_housing_height}"/>
+            </geometry>
+            <origin xyz="0 0 0" rpy="0 0 0"/>
+            <material name="black"/>
+        </visual>
+        <inertial>
+            <mass value="1.0"/>
+            <origin xyz="${link2_length/2} 0 0" rpy="0 0 0"/>
+            <inertia ixx="0.01" ixy="0" ixz="0" iyy="0.01" iyz="0" izz="0.01"/>
+        </inertial>
+    </link>
+    <joint name="joint3" type="revolute">
         <parent link="link2"/>
-        <child link="link3"/>
-        <origin xyz="0.4 0 0" rpy="0 0 0"/>
+        <child link="quill_housing_link"/>
+        <origin xyz="${link2_length} 0 0" rpy="0 0 0"/>
         <axis xyz="0 0 1"/>
-        <limit lower="0" upper="1.0" effort="10" velocity="1.0"/>
-    </joint>
-    <link name="link3">
-        <visual>
-            <geometry>
-                <cylinder length="0.5" radius="0.02"/>
-            </geometry>
-            <origin xyz="0 0 -0.25" rpy="0 0 0"/>
-        </visual>
-        <collision>
-            <geometry>
-                <cylinder length="0.5" radius="0.02"/>
-            </geometry>
-            <origin xyz="0 0 -0.25" rpy="0 0 0"/>
+        <limit lower="${-PI}" upper="${PI}" effort="50" velocity="2.0"/>
+    </joint>
+    <link name="quill_housing_link">
+        <visual>
+            <geometry>
+                <cylinder radius="${quill_housing_radius}" length="${quill_housing_length}"/>
+            </geometry>
+            <origin xyz="0 0 ${-quill_housing_length/4}" rpy="0 0 0"/>
+            <material name="light_grey"/>
+        </visual>
+        <collision>
+            <geometry>
+                <cylinder radius="${quill_housing_radius}" length="${quill_housing_length}"/>
+            </geometry>
+            <origin xyz="0 0 ${-quill_housing_length/4}" rpy="0 0 0"/>
+        </collision>
+        <inertial>
+            <mass value="0.5"/>
+            <inertia ixx="0.001" ixy="0" ixz="0" iyy="0.001" iyz="0" izz="0.001"/>
+        </inertial>
+    </link>
+    <joint name="joint4" type="prismatic">
+        <parent link="quill_housing_link"/>
+        <child link="tool_link"/>
+        <origin xyz="0 0 0" rpy="0 0 0"/>
+        <axis xyz="0 0 -1"/>
+        <limit lower="0.0" upper="0.15" effort="50" velocity="0.5"/>
+    </joint>
+    <link name="tool_link">
+        <visual>
+            <geometry>
+                <cylinder radius="${quill_radius}" length="${quill_length}"/>
+            </geometry>
+            <origin xyz="0 0 ${-quill_length/2}" rpy="0 0 0"/>
+            <material name="chrome"/>
+        </visual>
+        <collision>
+            <geometry>
+                <cylinder radius="${quill_radius}" length="${quill_length}"/>
+            </geometry>
+            <origin xyz="0 0 ${-quill_length/2}" rpy="0 0 0"/>
         </collision>
         <inertial>
             <mass value="0.2"/>
-            <inertia ixx="0.1" ixy="0" ixz="0" iyy="0.1" iyz="0" izz="0.1"/>
-        </inertial>
-    </link>
-    <joint name="joint4" type="revolute">
-        <parent link="link3"/>
-        <child link="end_effector_link"/>
-        <origin xyz="0 0 -0.5" rpy="0 0 0"/>
-        <axis xyz="0 0 1"/>
-        <limit lower="-3.14" upper="3.14" effort="10" velocity="1.0"/>
-    </joint>
-    <link name="end_effector_link">
-        <visual>
-            <geometry>
-                <box size="0.1 0.1 0.1"/>
-            </geometry>
-            <origin xyz="0 0 0" rpy="0 0 0"/>
-        </visual>
-        <collision>
-            <geometry>
-                <box size="0.1 0.1 0.1"/>
-            </geometry>
-            <origin xyz="0 0 0" rpy="0 0 0"/>
-        </collision>
-        <inertial>
-            <mass value="0.1"/>
-            <inertia ixx="0.1" ixy="0" ixz="0" iyy="0.1" iyz="0" izz="0.1"/>
-        </inertial>
-    </link>
+            <inertia ixx="0.001" ixy="0" ixz="0" iyy="0.001" iyz="0" izz="0.001"/>
+        </inertial>
+    </link>
+    <ros2_control name="GazeboSystem" type="system">
+        <hardware>
+            <plugin>gz_ros2_control/GazeboSimSystem</plugin>
+        </hardware>
+        <joint name="joint1">
+            <command_interface name="position"/>
+            <state_interface name="position"/>
+            <state_interface name="velocity"/>
+        </joint>
+        <joint name="joint2">
+            <command_interface name="position"/>
+            <state_interface name="position"/>
+            <state_interface name="velocity"/>
+        </joint>
+        <joint name="joint3">
+            <command_interface name="position"/>
+            <state_interface name="position"/>
+            <state_interface name="velocity"/>
+        </joint>
+        <joint name="joint4">
+            <command_interface name="position"/>
+            <state_interface name="position"/>
+            <state_interface name="velocity"/>
+        </joint>
+    </ros2_control>
+    <gazebo>
+        <plugin filename="gz_ros2_control-system" name="gz_ros2_control::GazeboSimROS2ControlPlugin">
+            <parameters>$(find scara_robot_simulation)/config/scara_controllers.yaml</parameters>
+        </plugin>
+    </gazebo>
 </robot>
