Commit message: fix: fix bot kinematics.
Signed-off-by: Paulo Santos <prms@ic.ufal.br>

File: src/scara_robot_simulation/description/urdf/scara_rrrp.ros2_control.xacro (robot description, xacro)
@@ -1,48 +1,52 @@
 <?xml version="1.0"?>
 <robot xmlns:xacro="http://www.ros.org/wiki/xacro" name="scara_rrrp">
-  <xacro:include filename="$(find scara_robot_simulation)/description/urdf/scara_rrrp.urdf.xacro" />
-  <ros2_control name="GazeboSystem" type="system">
-    <hardware>
-        <plugin>gz_ros2_control/GazeboSimSystem</plugin>
-    </hardware>
-    <joint name="joint1">
-      <command_interface name="position">
-        <param name="min">-3.14</param>
-        <param name="max">3.14</param>
-      </command_interface>
-      <state_interface name="position"/>
-      <state_interface name="velocity"/>
-    </joint>
-    <joint name="joint2">
-      <command_interface name="position">
-        <param name="min">-2.5</param>
-        <param name="max">2.5</param>
-      </command_interface>
-      <state_interface name="position"/>
-      <state_interface name="velocity"/>
-    </joint>
-    <joint name="joint3">
-      <command_interface name="position">
-        <param name="min">-3.14</param>
-        <param name="max">3.14</param>
-      </command_interface>
-      <state_interface name="position"/>
-      <state_interface name="velocity"/>
-    </joint>
-    <joint name="joint4">
-      <command_interface name="position">
-        <param name="min">0</param>
-        <param name="max">1.0</param>
-      </command_interface>
-      <state_interface name="position"/>
-      <state_interface name="velocity"/>
-    </joint>
-  </ros2_control>
-  <gazebo>
-      <plugin filename="gz_ros2_control-system" name="gz_ros2_control::GazeboSimROS2ControlPlugin">
-      <parameters>
-          $(find scara_robot_simulation)/config/scara_controllers.yaml
-      </parameters>
-    </plugin>
-  </gazebo>
+    <xacro:include filename="$(find scara_robot_simulation)/description/urdf/scara_rrrp.urdf.xacro"/>
+    <ros2_control name="GazeboSystem" type="system">
+        <hardware>
+            <plugin>gz_ros2_control/GazeboSimSystem</plugin>
+        </hardware>
+        # theta1
+        <joint name="joint1">
+            <command_interface name="position">
+                <param name="min">-3.14</param>
+                <param name="max">3.14</param>
+            </command_interface>
+            <state_interface name="position"/>
+            <state_interface name="velocity"/>
+        </joint>
+        # theta2
+        <joint name="joint2">
+            <command_interface name="position">
+                <param name="min">-2.9</param>
+                <param name="max">2.9</param>
+            </command_interface>
+            <state_interface name="position"/>
+            <state_interface name="velocity"/>
+        </joint>
+        # theta3
+        <joint name="joint3">
+            <command_interface name="position">
+                <param name="min">-3.14</param>
+                <param name="max">3.14</param>
+            </command_interface>
+            <state_interface name="position"/>
+            <state_interface name="velocity"/>
+        </joint>
+        # dz
+        <joint name="joint4">
+            <command_interface name="position">
+                <param name="min">-5.0</param>
+                <param name="max">5.0</param>
+            </command_interface>
+            <state_interface name="position"/>
+            <state_interface name="velocity"/>
+        </joint>
+    </ros2_control>
+    <gazebo>
+        <plugin filename="gz_ros2_control-system" name="gz_ros2_control::GazeboSimROS2ControlPlugin">
+            <parameters>
+                $(find scara_robot_simulation)/config/scara_controllers.yaml
+            </parameters>
+        </plugin>
+    </gazebo>
 </robot>

File: src/scara_robot_simulation/description/urdf/scara_rrrp.urdf.xacro (robot description, xacro)
@@ -10,7 +10,7 @@
     <xacro:property name="joint_housing_radius" value="0.03"/>
     <xacro:property name="joint_housing_height" value="0.12"/>
-    <xacro:property name="quill_housing_length" value="0.1"/>
+    <xacro:property name="quill_housing_length" value="0.05"/>
     <xacro:property name="quill_housing_radius" value="0.03"/>
-    <xacro:property name="quill_length" value="0.25"/>
+    <xacro:property name="quill_length" value="0.45"/>
     <xacro:property name="quill_radius" value="0.02"/>
     <material name="light_grey">
@@ -90,5 +90,5 @@
         <origin xyz="${link1_length} 0 0" rpy="0 0 0"/>
         <axis xyz="0 0 1"/>
-        <limit lower="${-PI*0.8}" upper="${PI*0.8}" effort="100" velocity="1.0"/>
+        <limit lower="${-PI*0.9}" upper="${PI*0.9}" effort="100" velocity="1.0"/>
     </joint>
     <link name="link2">
@@ -131,5 +131,5 @@
                 <cylinder radius="${quill_housing_radius}" length="${quill_housing_length}"/>
             </geometry>
-            <origin xyz="0 0 ${-quill_housing_length/4}" rpy="0 0 0"/>
+            <origin xyz="0 0 ${-quill_housing_length/2}" rpy="0 0 0"/>
             <material name="light_grey"/>
         </visual>
@@ -138,5 +138,5 @@
                 <cylinder radius="${quill_housing_radius}" length="${quill_housing_length}"/>
             </geometry>
-            <origin xyz="0 0 ${-quill_housing_length/4}" rpy="0 0 0"/>
+            <origin xyz="0 0 ${-quill_housing_length/2}" rpy="0 0 0"/>
         </collision>
         <inertial>
@@ -150,5 +150,5 @@
         <origin xyz="0 0 0" rpy="0 0 0"/>
         <axis xyz="0 0 -1"/>
-        <limit lower="0.0" upper="0.15" effort="50" velocity="0.5"/>
+        <limit lower="-5.0" upper="5.0" effort="50" velocity="0.5"/>
     </joint>
     <link name="tool_link">
@@ -171,33 +171,3 @@
         </inertial>
     </link>
-    <ros2_control name="GazeboSystem" type="system">
-        <hardware>
-            <plugin>gz_ros2_control/GazeboSimSystem</plugin>
-        </hardware>
-        <joint name="joint1">
-            <command_interface name="position"/>
-            <state_interface name="position"/>
-            <state_interface name="velocity"/>
-        </joint>
-        <joint name="joint2">
-            <command_interface name="position"/>
-            <state_interface name="position"/>
-            <state_interface name="velocity"/>
-        </joint>
-        <joint name="joint3">
-            <command_interface name="position"/>
-            <state_interface name="position"/>
-            <state_interface name="velocity"/>
-        </joint>
-        <joint name="joint4">
-            <command_interface name="position"/>
-            <state_interface name="position"/>
-            <state_interface name="velocity"/>
-        </joint>
-    </ros2_control>
-    <gazebo>
-        <plugin filename="gz_ros2_control-system" name="gz_ros2_control::GazeboSimROS2ControlPlugin">
-            <parameters>$(find scara_robot_simulation)/config/scara_controllers.yaml</parameters>
-        </plugin>
-    </gazebo>
 </robot>
